File: electronics/view_base/view_base.sch (KiCad schematic (older format))
At the start: 105 parts, among them J1 BLDC, J2 USB_C_Receptacle_USB2.0, J3 LCD, J4 A, J5 B, Q1 MMBT4403, Q2 UMH3N, U1 MT6701-CT, U2 T-Micro32_Plus, U3 CH340C, U4 HX711, U5 TMC6300, U6 AP2114HA-3.3, U7 SN74LV1T34DBV, U8 VEML7700

Commit message: Motor is available from SparkFun
Parts:
- Z10: AliExpress https://www.aliexpress.com/item/1005001384349991.html -> (none); Note (none) -> SparkFun: https://www.sparkfun.com/products/20441
Changed lines of the file:
@@
 F 2 "BOM_Only:bom_only_no_pin" H 8050 1800 60  0001 C CNN
 F 3 "" H 8050 1800 60  0001 C CNN
-F 4 "" H 8050 1800 50  0001 C CNN "Note"
-F 5 "https://www.aliexpress.com/item/1005001384349991.html" H 8050 1800 50  0001 C CNN "AliExpress"
+F 4 "SparkFun: https://www.sparkfun.com/products/20441" H 8050 1800 50  0001 C CNN "Note"
+F 5 "" H 8050 1800 50  0001 C CNN "AliExpress"
 	1    8050 1800
 	1    0    0    -1
